Commit message: Adding readme

File: gazebo/urdf/foxglove_box.urdf (robot description, URDF)
Before this commit: robot foxglove_block, 1 links, 0 joints
Links:
- link root_link: geometry collision box size=0.4 0.1 0.1; visual mesh filename=package://babbling_example/meshes/foxglove_box.dae scale=0.05 0.05 0.05

File: gazebo/urdf/kinect.urdf.xacro (robot description, xacro)
@@ -24,5 +24,5 @@
        <origin xyz="0 0 0" rpy="0 0 ${pi/2}"/>
         <geometry>
-         <mesh filename="package://fg_gazebo_example/meshes/kinect.dae"/>
+         <mesh filename="package://babbling_example/meshes/kinect.dae"/>
         </geometry>
       </visual>

File: gazebo/urdf/robot.xacro (robot description, xacro)
@@ -2,5 +2,5 @@
 <robot xmlns:xacro="http://wiki.ros.org/xacro" name="ur5e_robot">
   <xacro:include filename="$(find ur_gazebo)/urdf/ur_macro.xacro"/>
-  <xacro:include filename="$(find fg_gazebo_example)/urdf/kinect.urdf.xacro"/>
+  <xacro:include filename="$(find babbling_example)/urdf/kinect.urdf.xacro"/>
   <xacro:arg name="joint_limit_params" default=""/>
   <xacro:arg name="physical_params" default=""/>
